Commit message: Remove Gimbal

File: urdf/hku_m100.urdf.xacro (robot description, xacro)
@@ -1,5 +1,5 @@
 <?xml version="1.0"?>
 <robot name="hku_m100" xmlns:xacro="http://www.ros.org/wiki/xacro">
-    <xacro:include filename="$(find hku_m100_description)/urdf/hku_m100_base_with_gimbal.urdf.xacro" />
+    <xacro:include filename="$(find hku_m100_description)/urdf/hku_m100_base.urdf.xacro" />
     <xacro:hku_m100_base_macro />
 </robot>

File: urdf/hku_m100_base.urdf.xacro (robot description, xacro)
@@ -23,4 +23,6 @@
       </collision>
     </link>
+    <link name="dummy"/>
+    <!-- DEFINE SENSORS HERE -->
     <!-- Sonar height sensor -->
      <!--<xacro:sonar_sensor name="sonar" parent="base_link" ros_topic="sonar_height" update_rate="10" min_range="0.03" max_range="3.0" field_of_view="${40*pi/180}" ray_count="3">
