Commit message: Launch kinect

File: urdf/hku_m100_base.urdf.xacro (robot description, xacro)
@@ -4,4 +4,5 @@
   <!-- Main quadrotor link -->
   <xacro:macro name="hku_m100_base_macro">
+    <!-- <link name="dummy"/> -->
     <link name="base_link">
       <inertial>
@@ -23,5 +24,9 @@
       </collision>
     </link>
-    <link name="dummy"/>
+    <!--
+    <joint name="dummy_joint" type="fixed">
+      <parent link="dummy"/>
+      <child2 link="base_link"/>
+    </joint> -->
     <!-- DEFINE SENSORS HERE -->
     <!-- Sonar height sensor -->
